File: Hardware/MIKA/MIKA.kicad_sch (KiCad schematic)
At the start: 0 parts

Commit message: here ya go my fellas
Other:
- added sheet CM5 GPIO (CM5.kicad_sch)
- added sheet High Speed (high_speed.kicad_sch)
- added sheet Power Regulation (power_regulation.kicad_sch)
- added sheet SPI <-> CAN (SPI_CAN.kicad_sch)
- note added: "Connectors ------------- HDMI Ethernet USB-C 2.0 (Debug) USB A 3.0 (Camera)"
