File: Hardware/MIKA/MIKA.kicad_sch (KiCad schematic)
At the start: 0 parts

Commit message: bahasdf;ladjsfhadf boooooooooooshksa
Other:
- sheet SPI <-> CAN renamed SPI Peripherals
- sheet CM5 GPIO ports: added {IMU_SPI}; removed none
- sheet Power Regulation ports: added +12V_Telem; removed none
- sheet SPI Peripherals ports: added +12V_Telem, {IMU_SPI}; removed none
- note added: "Rate my schematic: 66/67"
