File: Hardware/MIKA/12VBuck.kicad_sch (KiCad schematic)
At the start: 14 parts, among them U1 LMR51635XDDCR

Commit message: ugahhghh might be layout time im a lil excited lwk
Parts:
- removed TP1: V_in_12V, TestPoint:TestPoint_THTPad_D3.0mm_Drill1.5mm, symbol Connector:TestPoint
- removed TP2: CB, TestPoint:TestPoint_THTPad_D3.0mm_Drill1.5mm, symbol Connector:TestPoint
- removed TP3: FB, TestPoint:TestPoint_THTPad_D3.0mm_Drill1.5mm, symbol Connector:TestPoint
- removed TP4: SW, TestPoint:TestPoint_THTPad_D3.0mm_Drill1.5mm, symbol Connector:TestPoint
- removed U1: LMR51635XDDCR, LHRS_ICs:DDC0006A-MFG, symbol 2026-04-25_18-34-12:LMR51635XDDCR
- added U1: LMR51635XDDCR, DDC0006A-MFG, symbol lhrs_power:LMR51635XDDCR
- L1: footprint LHRS_Passives:74439369082 -> LHRS_Power:XAL5050822MEC; LCSC P/N (none) -> C5309356; P/N 74439369082 -> XAL5050-822MEC
Connections:
- net CB: now also U1.6 (CB)
- net FB: now also U1.1 (FB)
- net GND: now also U1.4 (GND)
- net SW: now also U1.5 (SW)
- net Vin renamed V_in
- net V_in: now also U1.2 (EN), U1.3 (VIN)
- net Vout renamed V_out
Other:
- note added: "Vin: 4.6V to 60V"
- note removed: "Test Points"
