File: Hardware/MIKA/PowerProtection.kicad_sch (KiCad schematic)
At the start: 18 parts, among them IC1 LM74502DDFR, Q1 PSMN012-100YS, Q2 PSMN012-100YS

Commit message: ugahhghh might be layout time im a lil excited lwk
Parts:
- IC1: Manufacturer_Name Texas Instruments -> (none); Manufacturer_Part_Number LM74502DDFR -> (none); Mouser Part Number 595-LM74502DDFR -> (none); Mouser Price/Stock https://www.mouser.co.uk/ProductDetail/Texas-Instruments/LM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 -> (none)
- R1, R4, R5, R6, R7: symbol Device:R_US -> Device:R
- R3: symbol Device:R_US -> Device:R; Mouser Part Number 594-MCT06030C3309FP5 -> (none)
Other:
- note added: "Supp Battery Range: 10V-14.7V"
Changed lines of the file:
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@@
 		)
 	)
+	(text "Supp Battery Range:\n10V-14.7V"
+		(exclude_from_sim no)
+		(at 23.622 40.132 0)
+		(effects
+			(font
+				(size 1.27 1.27)
+			)
+		)
+	)
 	(text_box "Resistor Dividers"
 		(exclude_from_sim no)
@@
 		(instances
 			(project "MIKA"
-				(path "/66ea9e27-3ca5-4edd-a0db-1f3995e73e78/63cc9483-26fc-4cfe-88b4-a1a939222ea3/77edfde6-c89b-445e-95e4-9eff45b62586"
+				(path "/66ea9e27-3ca5-4edd-a0db-1f3995e73e78/63cc9483-26fc-4cfe-88b4-a1a939222ea3/59f3a675-0ec5-407b-bb19-7d9a2c9c96aa"
 					(reference "D1")
 					(unit 1)
@@
 		(instances
 			(project "MIKA"
-				(path "/66ea9e27-3ca5-4edd-a0db-1f3995e73e78/63cc9483-26fc-4cfe-88b4-a1a939222ea3/77edfde6-c89b-445e-95e4-9eff45b62586"
+				(path "/66ea9e27-3ca5-4edd-a0db-1f3995e73e78/63cc9483-26fc-4cfe-88b4-a1a939222ea3/59f3a675-0ec5-407b-bb19-7d9a2c9c96aa"
 					(reference "C3")
 					(unit 1)
@@
 		(instances
 			(project "MIKA"
-				(path "/66ea9e27-3ca5-4edd-a0db-1f3995e73e78/63cc9483-26fc-4cfe-88b4-a1a939222ea3/77edfde6-c89b-445e-95e4-9eff45b62586"
+				(path "/66ea9e27-3ca5-4edd-a0db-1f3995e73e78/63cc9483-26fc-4cfe-88b4-a1a939222ea3/59f3a675-0ec5-407b-bb19-7d9a2c9c96aa"
 					(reference "D2")
 					(unit 1)
@@
 	)
 	(symbol
-		(lib_id "Device:R_US")
+		(lib_id "Device:R")
 		(at 43.18 62.23 180)
 		(unit 1)
@@
 		(instances
 			(project "MIKA"
-				(path "/66ea9e27-3ca5-4edd-a0db-1f3995e73e78/63cc9483-26fc-4cfe-88b4-a1a939222ea3/77edfde6-c89b-445e-95e4-9eff45b62586"
+				(path "/66ea9e27-3ca5-4edd-a0db-1f3995e73e78/63cc9483-26fc-4cfe-88b4-a1a939222ea3/59f3a675-0ec5-407b-bb19-7d9a2c9c96aa"
 					(reference "R1")
 					(unit 1)
@@
 	)
 	(symbol
-		(lib_id "Device:R_US")
+		(lib_id "Device:R")
 		(at 139.7 90.17 180)
 		(unit 1)
@@
 		(instances
 			(project "MIKA"
-				(path "/66ea9e27-3ca5-4edd-a0db-1f3995e73e78/63cc9483-26fc-4cfe-88b4-a1a939222ea3/77edfde6-c89b-445e-95e4-9eff45b62586"
+				(path "/66ea9e27-3ca5-4edd-a0db-1f3995e73e78/63cc9483-26fc-4cfe-88b4-a1a939222ea3/59f3a675-0ec5-407b-bb19-7d9a2c9c96aa"
 					(reference "R6")
 					(unit 1)
@@
 		(instances
 			(project "MIKA"
-				(path "/66ea9e27-3ca5-4edd-a0db-1f3995e73e78/63cc9483-26fc-4cfe-88b4-a1a939222ea3/77edfde6-c89b-445e-95e4-9eff45b62586"
+				(path "/66ea9e27-3ca5-4edd-a0db-1f3995e73e78/63cc9483-26fc-4cfe-88b4-a1a939222ea3/59f3a675-0ec5-407b-bb19-7d9a2c9c96aa"
 					(reference "C1")
 					(unit 1)
@@
 	)
 	(symbol
-		(lib_id "Device:R_US")
+		(lib_id "Device:R")
 		(at 67.31 57.15 90)
 		(unit 1)
@@
 			)
 		)
-		(property "Mouser Part Number" "594-MCT06030C3309FP5 "
-			(at 67.31 57.15 0)
-			(hide yes)
-			(show_name no)
-			(do_not_autoplace no)
-			(effects
-				(font
-					(size 1.27 1.27)
-				)
-			)
-		)
 		(property "LCSC P/N" "C2074308"
 			(at 67.31 57.15 0)
@@
 		(instances
 			(project "MIKA"
-				(path "/66ea9e27-3ca5-4edd-a0db-1f3995e73e78/63cc9483-26fc-4cfe-88b4-a1a939222ea3/77edfde6-c89b-445e-95e4-9eff45b62586"
+				(path "/66ea9e27-3ca5-4edd-a0db-1f3995e73e78/63cc9483-26fc-4cfe-88b4-a1a939222ea3/59f3a675-0ec5-407b-bb19-7d9a2c9c96aa"
 					(reference "R3")
 					(unit 1)
@@
 			)
 		)
-		(property "Mouser Part Number" "595-LM74502DDFR"
-			(at 87.63 572.39 0)
-			(hide yes)
-			(show_name no)
-			(do_not_autoplace no)
-			(effects
-				(font
-					(size 1.27 1.27)
-				)
-				(justify left top)
-			)
-		)
-		(property "Mouser Price/Stock" "https://www.mouser.co.uk/ProductDetail/Texas-Instruments/LM74502HDDFR?qs=t7xnP681wgWDbfat8Yg%252B%2Fg%3D%3D"
-			(at 87.63 672.39 0)
-			(hide yes)
-			(show_name no)
-			(do_not_autoplace no)
-			(effects
-				(font
-					(size 1.27 1.27)
-				)
-				(justify left top)
-			)
-		)
-		(property "Manufacturer_Name" "Texas Instruments"
-			(at 87.63 772.39 0)
-			(hide yes)
-			(show_name no)
-			(do_not_autoplace no)
-			(effects
-				(font
-					(size 1.27 1.27)
-				)
-				(justify left top)
-			)
-		)
-		(property "Manufacturer_Part_Number" "LM74502DDFR"
-			(at 87.63 872.39 0)
-			(hide yes)
-			(show_name no)
-			(do_not_autoplace no)
-			(effects
-				(font
-					(size 1.27 1.27)
-				)
-				(justify left top)
-			)
-		)
 		(property "P/N" "LM74502DDFR"
 			(at 58.42 77.47 0)
@@
 		(instances
 			(project "MIKA"
-				(path "/66ea9e27-3ca5-4edd-a0db-1f3995e73e78/63cc9483-26fc-4cfe-88b4-a1a939222ea3/77edfde6-c89b-445e-95e4-9eff45b62586"
+				(path "/66ea9e27-3ca5-4edd-a0db-1f3995e73e78/63cc9483-26fc-4cfe-88b4-a1a939222ea3/59f3a675-0ec5-407b-bb19-7d9a2c9c96aa"
 					(reference "IC1")
 					(unit 1)
@@
 			)
 		)
-		(property "Sim.Device" "NMOS"
-			(at 73.025 46.99 0)
-			(hide yes)
-			(show_name no)
-			(do_not_autoplace no)
-			(effects
-				(font
-					(size 1.27 1.27)
-				)
-			)
-		)
-		(property "Sim.Type" "VDMOS"
-			(at 74.93 46.99 0)
-			(hide yes)
-			(show_name no)
-			(do_not_autoplace no)
-			(effects
-				(font
-					(size 1.27 1.27)
-				)
-			)
-		)
-		(property "Sim.Pins" "1=D 2=G 3=S"
-			(at 71.12 46.99 0)
-			(hide yes)
-			(show_name no)
-			(do_not_autoplace no)
-			(effects
-				(font
-					(size 1.27 1.27)
-				)
-			)
-		)
 		(property "P/N" "PSMN012-100YSFX"
 			(at 55.88 46.99 0)
@@
 		(instances
 			(project "MIKA"
-				(path "/66ea9e27-3ca5-4edd-a0db-1f3995e73e78/63cc9483-26fc-4cfe-88b4-a1a939222ea3/77edfde6-c89b-445e-95e4-9eff45b62586"
+				(path "/66ea9e27-3ca5-4edd-a0db-1f3995e73e78/63cc9483-26fc-4cfe-88b4-a1a939222ea3/59f3a675-0ec5-407b-bb19-7d9a2c9c96aa"
 					(reference "Q1")
 					(unit 1)
@@
 		(instances
 			(project "MIKA"
-				(path "/66ea9e27-3ca5-4edd-a0db-1f3995e73e78/63cc9483-26fc-4cfe-88b4-a1a939222ea3/77edfde6-c89b-445e-95e4-9eff45b62586"
+				(path "/66ea9e27-3ca5-4edd-a0db-1f3995e73e78/63cc9483-26fc-4cfe-88b4-a1a939222ea3/59f3a675-0ec5-407b-bb19-7d9a2c9c96aa"
 					(reference "C6")
 					(unit 1)
@@
 		(instances
 			(project "MIKA"
-				(path "/66ea9e27-3ca5-4edd-a0db-1f3995e73e78/63cc9483-26fc-4cfe-88b4-a1a939222ea3/77edfde6-c89b-445e-95e4-9eff45b62586"
+				(path "/66ea9e27-3ca5-4edd-a0db-1f3995e73e78/63cc9483-26fc-4cfe-88b4-a1a939222ea3/59f3a675-0ec5-407b-bb19-7d9a2c9c96aa"
 					(reference "C4")
 					(unit 1)
@@
 		(instances
 			(project "MIKA"
-				(path "/66ea9e27-3ca5-4edd-a0db-1f3995e73e78/63cc9483-26fc-4cfe-88b4-a1a939222ea3/77edfde6-c89b-445e-95e4-9eff45b62586"
+				(path "/66ea9e27-3ca5-4edd-a0db-1f3995e73e78/63cc9483-26fc-4cfe-88b4-a1a939222ea3/59f3a675-0ec5-407b-bb19-7d9a2c9c96aa"
 					(reference "C5")
 					(unit 1)
@@
 			)
 		)
-		(property "Sim.Device" "NMOS"
-			(at 76.835 46.99 0)
-			(hide yes)
-			(show_name no)
-			(do_not_autoplace no)
-			(effects
-				(font
-					(size 1.27 1.27)
-				)
-			)
-		)
-		(property "Sim.Type" "VDMOS"
-			(at 74.93 46.99 0)
-			(hide yes)
-			(show_name no)
-			(do_not_autoplace no)
-			(effects
-				(font
-					(size 1.27 1.27)
-				)
-			)
-		)
-		(property "Sim.Pins" "1=D 2=G 3=S"
-			(at 78.74 46.99 0)
-			(hide yes)
-			(show_name no)
-			(do_not_autoplace no)
-			(effects
-				(font
-					(size 1.27 1.27)
-				)
-			)
-		)
 		(property "P/N" "PSMN012-100YSFX"
 			(at 93.98 46.99 0)
@@
 		(instances
 			(project "MIKA"
-				(path "/66ea9e27-3ca5-4edd-a0db-1f3995e73e78/63cc9483-26fc-4cfe-88b4-a1a939222ea3/77edfde6-c89b-445e-95e4-9eff45b62586"
+				(path "/66ea9e27-3ca5-4edd-a0db-1f3995e73e78/63cc9483-26fc-4cfe-88b4-a1a939222ea3/59f3a675-0ec5-407b-bb19-7d9a2c9c96aa"
 					(reference "Q2")
 					(unit 1)
@@
 	)
 	(symbol
-		(lib_id "Device:R_US")
+		(lib_id "Device:R")
 		(at 120.65 90.17 0)
 		(unit 1)
@@
 		(instances
 			(project "MIKA"
-				(path "/66ea9e27-3ca5-4edd-a0db-1f3995e73e78/63cc9483-26fc-4cfe-88b4-a1a939222ea3/77edfde6-c89b-445e-95e4-9eff45b62586"
+				(path "/66ea9e27-3ca5-4edd-a0db-1f3995e73e78/63cc9483-26fc-4cfe-88b4-a1a939222ea3/59f3a675-0ec5-407b-bb19-7d9a2c9c96aa"
 					(reference "R5")
 					(unit 1)
@@
 		(instances
 			(project "MIKA"
-				(path "/66ea9e27-3ca5-4edd-a0db-1f3995e73e78/63cc9483-26fc-4cfe-88b4-a1a939222ea3/77edfde6-c89b-445e-95e4-9eff45b62586"
+				(path "/66ea9e27-3ca5-4edd-a0db-1f3995e73e78/63cc9483-26fc-4cfe-88b4-a1a939222ea3/59f3a675-0ec5-407b-bb19-7d9a2c9c96aa"
 					(reference "C2")
 					(unit 1)
@@
 		(instances
 			(project "MIKA"
-				(path "/66ea9e27-3ca5-4edd-a0db-1f3995e73e78/63cc9483-26fc-4cfe-88b4-a1a939222ea3/77edfde6-c89b-445e-95e4-9eff45b62586"
+				(path "/66ea9e27-3ca5-4edd-a0db-1f3995e73e78/63cc9483-26fc-4cfe-88b4-a1a939222ea3/59f3a675-0ec5-407b-bb19-7d9a2c9c96aa"
 					(reference "C7")
 					(unit 1)
@@
 	)
 	(symbol
-		(lib_id "Device:R_US")
+		(lib_id "Device:R")
 		(at 115.57 77.47 0)
 		(unit 1)
@@
 		(instances
 			(project "MIKA"
-				(path "/66ea9e27-3ca5-4edd-a0db-1f3995e73e78/63cc9483-26fc-4cfe-88b4-a1a939222ea3/77edfde6-c89b-445e-95e4-9eff45b62586"
+				(path "/66ea9e27-3ca5-4edd-a0db-1f3995e73e78/63cc9483-26fc-4cfe-88b4-a1a939222ea3/59f3a675-0ec5-407b-bb19-7d9a2c9c96aa"
 					(reference "R4")
 					(unit 1)
@@
 	)
 	(symbol
-		(lib_id "Device:R_US")
+		(lib_id "Device:R")
 		(at 134.62 77.47 0)
 		(unit 1)
@@
 		(instances
 			(project "MIKA"
-				(path "/66ea9e27-3ca5-4edd-a0db-1f3995e73e78/63cc9483-26fc-4cfe-88b4-a1a939222ea3/77edfde6-c89b-445e-95e4-9eff45b62586"
+				(path "/66ea9e27-3ca5-4edd-a0db-1f3995e73e78/63cc9483-26fc-4cfe-88b4-a1a939222ea3/59f3a675-0ec5-407b-bb19-7d9a2c9c96aa"
 					(reference "R7")
 					(unit 1)

Commit message: bahasdf;ladjsfhadf boooooooooooshksa
Parts:
- renumbered C5 to C10, C6 to C11, C7 to C12, C1 to C6, C2 to C7, C3 to C8, C4 to C9, D2 to D6, D1 to D7, R4 to R10, R5 to R11, R7 to R12, R6 to R13, R1 to R8, R3 to R9
Changed lines of the file:
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@@
 		(in_pos_files yes)
 		(dnp no)
-		(property "Reference" "D1"
+		(property "Reference" "D7"
 			(at 40.64 82.296 0)
 			(show_name no)
@@
 			(project "MIKA"
 				(path "/66ea9e27-3ca5-4edd-a0db-1f3995e73e78/63cc9483-26fc-4cfe-88b4-a1a939222ea3/59f3a675-0ec5-407b-bb19-7d9a2c9c96aa"
-					(reference "D1")
+					(reference "D7")
 					(unit 1)
 				)
@@
 		(dnp no)
 		(fields_autoplaced yes)
-		(property "Reference" "C3"
+		(property "Reference" "C8"
 			(at 57.785 80.0099 0)
 			(show_name no)
@@
 			(project "MIKA"
 				(path "/66ea9e27-3ca5-4edd-a0db-1f3995e73e78/63cc9483-26fc-4cfe-88b4-a1a939222ea3/59f3a675-0ec5-407b-bb19-7d9a2c9c96aa"
-					(reference "C3")
+					(reference "C8")
 					(unit 1)
 				)
@@
 		(in_pos_files yes)
 		(dnp no)
-		(property "Reference" "D2"
+		(property "Reference" "D6"
 			(at 22.606 49.276 0)
 			(show_name no)
@@
 			(project "MIKA"
 				(path "/66ea9e27-3ca5-4edd-a0db-1f3995e73e78/63cc9483-26fc-4cfe-88b4-a1a939222ea3/59f3a675-0ec5-407b-bb19-7d9a2c9c96aa"
-					(reference "D2")
+					(reference "D6")
 					(unit 1)
 				)
@@
 		(dnp no)
 		(fields_autoplaced yes)
-		(property "Reference" "R1"
+		(property "Reference" "R8"
 			(at 45.72 60.9599 0)
 			(show_name no)
@@
 			(project "MIKA"
 				(path "/66ea9e27-3ca5-4edd-a0db-1f3995e73e78/63cc9483-26fc-4cfe-88b4-a1a939222ea3/59f3a675-0ec5-407b-bb19-7d9a2c9c96aa"
-					(reference "R1")
+					(reference "R8")
 					(unit 1)
 				)
@@
 		(in_pos_files yes)
 		(dnp no)
-		(property "Reference" "R6"
+		(property "Reference" "R13"
 			(at 137.668 90.17 90)
 			(show_name no)
@@
 			(project "MIKA"
 				(path "/66ea9e27-3ca5-4edd-a0db-1f3995e73e78/63cc9483-26fc-4cfe-88b4-a1a939222ea3/59f3a675-0ec5-407b-bb19-7d9a2c9c96aa"
-					(reference "R6")
+					(reference "R13")
 					(unit 1)
 				)
@@
 		(in_pos_files yes)
 		(dnp no)
-		(property "Reference" "C1"
+		(property "Reference" "C6"
 			(at 38.1 49.5299 0)
 			(show_name no)
@@
 			(project "MIKA"
 				(path "/66ea9e27-3ca5-4edd-a0db-1f3995e73e78/63cc9483-26fc-4cfe-88b4-a1a939222ea3/59f3a675-0ec5-407b-bb19-7d9a2c9c96aa"
-					(reference "C1")
+					(reference "C6")
 					(unit 1)
 				)
@@
 		(in_pos_files yes)
 		(dnp no)
-		(property "Reference" "R3"
+		(property "Reference" "R9"
 			(at 67.31 54.61 90)
 			(show_name no)
@@
 			(project "MIKA"
 				(path "/66ea9e27-3ca5-4edd-a0db-1f3995e73e78/63cc9483-26fc-4cfe-88b4-a1a939222ea3/59f3a675-0ec5-407b-bb19-7d9a2c9c96aa"
-					(reference "R3")
+					(reference "R9")
 					(unit 1)
 				)
@@
 		(in_pos_files yes)
 		(dnp no)
-		(property "Reference" "C6"
+		(property "Reference" "C11"
 			(at 113.284 89.154 0)
 			(show_name no)
@@
 			(project "MIKA"
 				(path "/66ea9e27-3ca5-4edd-a0db-1f3995e73e78/63cc9483-26fc-4cfe-88b4-a1a939222ea3/59f3a675-0ec5-407b-bb19-7d9a2c9c96aa"
-					(reference "C6")
+					(reference "C11")
 					(unit 1)
 				)
@@
 		(in_pos_files yes)
 		(dnp no)
-		(property "Reference" "C4"
+		(property "Reference" "C9"
 			(at 54.864 62.23 0)
 			(show_name no)
@@
 			(project "MIKA"
 				(path "/66ea9e27-3ca5-4edd-a0db-1f3995e73e78/63cc9483-26fc-4cfe-88b4-a1a939222ea3/59f3a675-0ec5-407b-bb19-7d9a2c9c96aa"
-					(reference "C4")
+					(reference "C9")
 					(unit 1)
 				)
@@
 		(in_pos_files yes)
 		(dnp no)
-		(property "Reference" "C5"
+		(property "Reference" "C10"
 			(at 112.395 49.5299 0)
 			(show_name no)
@@
 			(project "MIKA"
 				(path "/66ea9e27-3ca5-4edd-a0db-1f3995e73e78/63cc9483-26fc-4cfe-88b4-a1a939222ea3/59f3a675-0ec5-407b-bb19-7d9a2c9c96aa"
-					(reference "C5")
+					(reference "C10")
 					(unit 1)
 				)
@@
 		(in_pos_files yes)
 		(dnp no)
-		(property "Reference" "R5"
+		(property "Reference" "R11"
 			(at 118.618 90.424 90)
 			(show_name no)
@@
 			(project "MIKA"
 				(path "/66ea9e27-3ca5-4edd-a0db-1f3995e73e78/63cc9483-26fc-4cfe-88b4-a1a939222ea3/59f3a675-0ec5-407b-bb19-7d9a2c9c96aa"
-					(reference "R5")
+					(reference "R11")
 					(unit 1)
 				)
@@
 		(in_pos_files yes)
 		(dnp no)
-		(property "Reference" "C2"
+		(property "Reference" "C7"
 			(at 31.75 82.5499 0)
 			(show_name no)
@@
 			(project "MIKA"
 				(path "/66ea9e27-3ca5-4edd-a0db-1f3995e73e78/63cc9483-26fc-4cfe-88b4-a1a939222ea3/59f3a675-0ec5-407b-bb19-7d9a2c9c96aa"
-					(reference "C2")
+					(reference "C7")
 					(unit 1)
 				)
@@
 		(in_pos_files yes)
 		(dnp no)
-		(property "Reference" "C7"
+		(property "Reference" "C12"
 			(at 132.08 88.9 0)
 			(show_name no)
@@
 			(project "MIKA"
 				(path "/66ea9e27-3ca5-4edd-a0db-1f3995e73e78/63cc9483-26fc-4cfe-88b4-a1a939222ea3/59f3a675-0ec5-407b-bb19-7d9a2c9c96aa"
-					(reference "C7")
+					(reference "C12")
 					(unit 1)
 				)
@@
 		(in_pos_files yes)
 		(dnp no)
-		(property "Reference" "R4"
+		(property "Reference" "R10"
 			(at 118.11 78.74 90)
 			(show_name no)
@@
 			(project "MIKA"
 				(path "/66ea9e27-3ca5-4edd-a0db-1f3995e73e78/63cc9483-26fc-4cfe-88b4-a1a939222ea3/59f3a675-0ec5-407b-bb19-7d9a2c9c96aa"
-					(reference "R4")
+					(reference "R10")
 					(unit 1)
 				)
@@
 		(in_pos_files yes)
 		(dnp no)
-		(property "Reference" "R7"
+		(property "Reference" "R12"
 			(at 137.16 77.47 90)
 			(show_name no)
@@
 			(project "MIKA"
 				(path "/66ea9e27-3ca5-4edd-a0db-1f3995e73e78/63cc9483-26fc-4cfe-88b4-a1a939222ea3/59f3a675-0ec5-407b-bb19-7d9a2c9c96aa"
-					(reference "R7")
-					(unit 1)
-				)
+					(reference "R12")
+					(unit 1)
+				)
