File: Hardware/MIKA/Power_Mux.kicad_sch (KiCad schematic)
At the start: 6 parts, among them U1 TPS2117DRLR

Commit message: ugahhghh might be layout time im a lil excited lwk
Parts:
- C1, C2, C3, C4: value 0.1uF -> 0.1u; Mfg MLASH168SB7104KTNA01 -> (none)
- U1: MANUFACTURER Texas Instruments -> (none); MAXIMUM_PACKAGE_HEIGHT 0.6mm -> (none); PARTREV A -> (none); STANDARD IPC-7351B -> (none)
Changed lines of the file:
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@@
 			)
 		)
-		(property "Value" "0.1uF"
+		(property "Value" "0.1u"
 			(at 91.8972 59.563 0)
 			(show_name no)
@@
 			)
 		)
-		(property "Mfg" "MLASH168SB7104KTNA01"
-			(at 88.9 58.42 0)
-			(hide yes)
-			(show_name no)
-			(do_not_autoplace no)
-			(effects
-				(font
-					(size 1.27 1.27)
-				)
-			)
-		)
 		(pin "1"
 		)
@@
 		(instances
 			(project "MIKA"
-				(path "/66ea9e27-3ca5-4edd-a0db-1f3995e73e78/63cc9483-26fc-4cfe-88b4-a1a939222ea3/bbd4617a-c7a2-42c0-8202-948d9fb46b7b"
+				(path "/66ea9e27-3ca5-4edd-a0db-1f3995e73e78/63cc9483-26fc-4cfe-88b4-a1a939222ea3/b25c6fa0-ff35-478e-9151-e00f6f5c12b7"
 					(reference "C4")
 					(unit 1)
 				)
 			)
-			(project "power-mux-block"
+			(project "Power_Mux"
 				(path "/c8207045-8aef-4538-bcc4-1e380c549c2c"
 					(reference "C4")
@@
 		(instances
 			(project "MIKA"
-				(path "/66ea9e27-3ca5-4edd-a0db-1f3995e73e78/63cc9483-26fc-4cfe-88b4-a1a939222ea3/bbd4617a-c7a2-42c0-8202-948d9fb46b7b"
+				(path "/66ea9e27-3ca5-4edd-a0db-1f3995e73e78/63cc9483-26fc-4cfe-88b4-a1a939222ea3/b25c6fa0-ff35-478e-9151-e00f6f5c12b7"
 					(reference "R1")
 					(unit 1)
 				)
 			)
-			(project "power-mux-block"
+			(project "Power_Mux"
 				(path "/c8207045-8aef-4538-bcc4-1e380c549c2c"
 					(reference "R1")
@@
 			)
 		)
-		(property "Value" "0.1uF"
+		(property "Value" "0.1u"
 			(at 24.5872 46.863 0)
 			(show_name no)
@@
 			)
 		)
-		(property "Mfg" "MLASH168SB7104KTNA01"
-			(at 21.59 45.72 0)
-			(hide yes)
-			(show_name no)
-			(do_not_autoplace no)
-			(effects
-				(font
-					(size 1.27 1.27)
-				)
-			)
-		)
 		(pin "1"
 		)
@@
 		(instances
 			(project "MIKA"
-				(path "/66ea9e27-3ca5-4edd-a0db-1f3995e73e78/63cc9483-26fc-4cfe-88b4-a1a939222ea3/bbd4617a-c7a2-42c0-8202-948d9fb46b7b"
+				(path "/66ea9e27-3ca5-4edd-a0db-1f3995e73e78/63cc9483-26fc-4cfe-88b4-a1a939222ea3/b25c6fa0-ff35-478e-9151-e00f6f5c12b7"
 					(reference "C1")
 					(unit 1)
 				)
 			)
-			(project "power-mux-block"
+			(project "Power_Mux"
 				(path "/c8207045-8aef-4538-bcc4-1e380c549c2c"
 					(reference "C1")
@@
 			)
 		)
-		(property "PARTREV" "A"
-			(at 60.96 62.23 0)
-			(hide yes)
-			(show_name no)
-			(do_not_autoplace no)
-			(effects
-				(font
-					(size 1.27 1.27)
-				)
-				(justify bottom)
-			)
-		)
-		(property "STANDARD" "IPC-7351B"
-			(at 60.96 62.23 0)
-			(hide yes)
-			(show_name no)
-			(do_not_autoplace no)
-			(effects
-				(font
-					(size 1.27 1.27)
-				)
-				(justify bottom)
-			)
-		)
-		(property "MAXIMUM_PACKAGE_HEIGHT" "0.6mm"
-			(at 60.96 62.23 0)
-			(hide yes)
-			(show_name no)
-			(do_not_autoplace no)
-			(effects
-				(font
-					(size 1.27 1.27)
-				)
-				(justify bottom)
-			)
-		)
-		(property "MANUFACTURER" "Texas Instruments"
-			(at 60.96 62.23 0)
-			(hide yes)
-			(show_name no)
-			(do_not_autoplace no)
-			(effects
-				(font
-					(size 1.27 1.27)
-				)
-				(justify bottom)
-			)
-		)
 		(property "P/N" "TPS2117DRLR"
 			(at 60.96 49.53 0)
@@
 		(instances
 			(project "MIKA"
-				(path "/66ea9e27-3ca5-4edd-a0db-1f3995e73e78/63cc9483-26fc-4cfe-88b4-a1a939222ea3/bbd4617a-c7a2-42c0-8202-948d9fb46b7b"
+				(path "/66ea9e27-3ca5-4edd-a0db-1f3995e73e78/63cc9483-26fc-4cfe-88b4-a1a939222ea3/b25c6fa0-ff35-478e-9151-e00f6f5c12b7"
 					(reference "U1")
 					(unit 1)
 				)
 			)
-			(project ""
+			(project "Power_Mux"
 				(path "/c8207045-8aef-4538-bcc4-1e380c549c2c"
 					(reference "U1")
@@
 			)
 		)
-		(property "Value" "0.1uF"
+		(property "Value" "0.1u"
 			(at 42.3672 69.723 0)
 			(show_name no)
@@
 			)
 		)
-		(property "Mfg" "MLASH168SB7104KTNA01"
-			(at 39.37 68.58 0)
-			(hide yes)
-			(show_name no)
-			(do_not_autoplace no)
-			(effects
-				(font
-					(size 1.27 1.27)
-				)
-			)
-		)
 		(pin "1"
 		)
@@
 		(instances
 			(project "MIKA"
-				(path "/66ea9e27-3ca5-4edd-a0db-1f3995e73e78/63cc9483-26fc-4cfe-88b4-a1a939222ea3/bbd4617a-c7a2-42c0-8202-948d9fb46b7b"
+				(path "/66ea9e27-3ca5-4edd-a0db-1f3995e73e78/63cc9483-26fc-4cfe-88b4-a1a939222ea3/b25c6fa0-ff35-478e-9151-e00f6f5c12b7"
 					(reference "C3")
 					(unit 1)
 				)
 			)
-			(project "power-mux-block"
+			(project "Power_Mux"
 				(path "/c8207045-8aef-4538-bcc4-1e380c549c2c"
 					(reference "C3")
@@
 			)
 		)
-		(property "Value" "0.1uF"
+		(property "Value" "0.1u"
 			(at 38.5572 46.863 0)
 			(show_name no)
@@
 			)
 		)
-		(property "Mfg" "MLASH168SB7104KTNA01"
-			(at 35.56 45.72 0)
-			(hide yes)
-			(show_name no)
-			(do_not_autoplace no)
-			(effects
-				(font
-					(size 1.27 1.27)
-				)
-			)
-		)
 		(pin "1"
 		)
@@
 		(instances
 			(project "MIKA"
-				(path "/66ea9e27-3ca5-4edd-a0db-1f3995e73e78/63cc9483-26fc-4cfe-88b4-a1a939222ea3/bbd4617a-c7a2-42c0-8202-948d9fb46b7b"
+				(path "/66ea9e27-3ca5-4edd-a0db-1f3995e73e78/63cc9483-26fc-4cfe-88b4-a1a939222ea3/b25c6fa0-ff35-478e-9151-e00f6f5c12b7"
 					(reference "C2")
 					(unit 1)
 				)
 			)
-			(project "power-mux-block"
+			(project "Power_Mux"
 				(path "/c8207045-8aef-4538-bcc4-1e380c549c2c"
 					(reference "C2")

Commit message: bahasdf;ladjsfhadf boooooooooooshksa
Parts:
- renumbered C1 to C31, C2 to C32, C3 to C33, C4 to C34, R1 to R21, U1 to U2
Changed lines of the file:
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@@
 		(in_pos_files yes)
 		(dnp no)
-		(property "Reference" "C4"
+		(property "Reference" "C34"
 			(at 91.8972 57.2516 0)
 			(show_name no)
@@
 			(project "MIKA"
 				(path "/66ea9e27-3ca5-4edd-a0db-1f3995e73e78/63cc9483-26fc-4cfe-88b4-a1a939222ea3/b25c6fa0-ff35-478e-9151-e00f6f5c12b7"
-					(reference "C4")
+					(reference "C34")
 					(unit 1)
 				)
@@
 		(in_pos_files yes)
 		(dnp no)
-		(property "Reference" "R1"
+		(property "Reference" "R21"
 			(at 78.994 67.564 0)
 			(show_name no)
@@
 			(project "MIKA"
 				(path "/66ea9e27-3ca5-4edd-a0db-1f3995e73e78/63cc9483-26fc-4cfe-88b4-a1a939222ea3/b25c6fa0-ff35-478e-9151-e00f6f5c12b7"
-					(reference "R1")
+					(reference "R21")
 					(unit 1)
 				)
@@
 		(in_pos_files yes)
 		(dnp no)
-		(property "Reference" "C1"
+		(property "Reference" "C31"
 			(at 24.5872 44.5516 0)
 			(show_name no)
@@
 			(project "MIKA"
 				(path "/66ea9e27-3ca5-4edd-a0db-1f3995e73e78/63cc9483-26fc-4cfe-88b4-a1a939222ea3/b25c6fa0-ff35-478e-9151-e00f6f5c12b7"
-					(reference "C1")
+					(reference "C31")
 					(unit 1)
 				)
@@
 		(dnp no)
 		(fields_autoplaced yes)
-		(property "Reference" "U1"
+		(property "Reference" "U2"
 			(at 60.96 44.45 0)
 			(show_name no)
@@
 			(project "MIKA"
 				(path "/66ea9e27-3ca5-4edd-a0db-1f3995e73e78/63cc9483-26fc-4cfe-88b4-a1a939222ea3/b25c6fa0-ff35-478e-9151-e00f6f5c12b7"
-					(reference "U1")
+					(reference "U2")
 					(unit 1)
 				)
@@
 		(in_pos_files yes)
 		(dnp no)
-		(property "Reference" "C3"
+		(property "Reference" "C33"
 			(at 42.3672 67.4116 0)
 			(show_name no)
@@
 			(project "MIKA"
 				(path "/66ea9e27-3ca5-4edd-a0db-1f3995e73e78/63cc9483-26fc-4cfe-88b4-a1a939222ea3/b25c6fa0-ff35-478e-9151-e00f6f5c12b7"
-					(reference "C3")
+					(reference "C33")
 					(unit 1)
 				)
@@
 		(in_pos_files yes)
 		(dnp no)
-		(property "Reference" "C2"
+		(property "Reference" "C32"
 			(at 38.5572 44.5516 0)
 			(show_name no)
@@
 			(project "MIKA"
 				(path "/66ea9e27-3ca5-4edd-a0db-1f3995e73e78/63cc9483-26fc-4cfe-88b4-a1a939222ea3/b25c6fa0-ff35-478e-9151-e00f6f5c12b7"
-					(reference "C2")
-					(unit 1)
-				)
+					(reference "C32")
+					(unit 1)
+				)
