File: Hardware/MIKA/SPI_CAN.kicad_sch (KiCad schematic)
At the start: 35 parts

Commit message: ugahhghh might be layout time im a lil excited lwk
Parts:
- removed C? (x2): 0.1uF, symbol Device:C
- removed C? (x2): 100nF, symbol Device:C
- removed C? (x2): 10uF, symbol Device:C
- added C? (x4): 0.1u, symbol Device:C
- added C?: 10uF, symbol Device:C
- added C?: 10u, symbol Device:C
- C22, C23, C24, C25: renamed from C?; value 10pF -> 10p
- C28, C29: renamed from C?; value 300nF -> 300n
- C30: renamed from C?; value 10uF -> 10u
- C32, C36: renamed from C?; value 0.1uF -> 0.1u
- gave numbers to parts that had none: 20
Connections:
- net +12V: now also C?.2, C?.2
- net +3.3V: now also C?.2, C?.2
- net GND: now also C?.1, C?.1, C?.1, C?.1, C?.1, C?.1
- net at U5.16 (V_{CCFLTR}): now also C?.2
- net at U4.16 (V_{CCFLTR}): now also C?.2

Commit message: bahasdf;ladjsfhadf boooooooooooshksa
Parts:
- removed C22, C23, C24, C25: 10p, symbol Device:C
- removed C28, C29: 300n, symbol Device:C
- removed C30, C?: 10u, symbol Device:C
- removed C32, C36, C? (x4): 0.1u, symbol Device:C
- removed C34, C?: 10uF, symbol Device:C
- removed D5, D6: LED, symbol Device:LED
- removed F6: Fuse, symbol Device:Fuse
- removed R16, R17: R, symbol Device:R
- removed U4, U5: TCAN4551RGYRQ1, Package_DFN_QFN:Texas_RGY_R-PVQFN-N20_EP2.05x3.05mm, symbol Interface_CAN_LIN:TCAN4551RGYRQ1
- removed Y1: 7M40000005, symbol Device:Crystal_GND24
- removed Y2: Crystal_GND24, symbol Device:Crystal_GND24
- added R39, R40: 22, symbol Device:R
- renumbered J9 to J12, J8 to J7, J7 to J8, J6 to J9, R19 to R35, R20 to R36, R18 to R37, R21 to R38
Connections:
- net C_SDO: now also R39.1
- net T_SDO: now also R40.1
- new net SPI <-> CarCAN/SDO: R39.2
- new net SPI <-> TelemCAN/SDO: R40.2
- no-connect marks 6 -> 0
Other:
- added sheet IMUs (IMUs.kicad_sch)
- added sheet SPI <-> CarCAN (spi_2_can.kicad_sch)
- added sheet SPI <-> TelemCAN (spi_2_can.kicad_sch)
- note removed: "40MHz External Crystal"
- note removed: "SPI <-> CarCAN"
- note removed: "SPI <-> TelemetryCAN"
- note removed: "Test Points"
- note removed: "use nINT for CAN fault detection"
- moved on the sheet: J10, J11, J12, J7, J8, J9, R35, R36, R37, R38
