File: Hardware/MIKA/USB-C_Connector.kicad_sch (KiCad schematic)
At the start: 8 parts, among them J1 USB_C_Receptacle_USB2.0_16P

Commit message: ugahhghh might be layout time im a lil excited lwk
Parts:
- C38: renamed from C?; value 4.7nF -> 4.7n
- gave numbers to parts that had none: 1
- renumbered C1 to C39, D1 to D7, D3 to D8, J1 to J12, R1 to R23, R2 to R24
Changed lines of the file:
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@@
 		(in_pos_files yes)
 		(dnp no)
-		(property "Reference" "R1"
+		(property "Reference" "R23"
 			(at 86.106 48.26 90)
 			(show_name no)
@@
 			(project "MIKA"
 				(path "/66ea9e27-3ca5-4edd-a0db-1f3995e73e78/c2d6fcaf-19aa-4c33-838f-5e0ce95c1959/7dc4223e-0f41-465d-891f-db8b5b137845"
-					(reference "R1")
+					(reference "R23")
 					(unit 1)
 				)
@@
 		(in_pos_files yes)
 		(dnp no)
-		(property "Reference" "R2"
+		(property "Reference" "R24"
 			(at 93.726 48.26 90)
 			(show_name no)
@@
 			(project "MIKA"
 				(path "/66ea9e27-3ca5-4edd-a0db-1f3995e73e78/c2d6fcaf-19aa-4c33-838f-5e0ce95c1959/7dc4223e-0f41-465d-891f-db8b5b137845"
-					(reference "R2")
+					(reference "R24")
 					(unit 1)
 				)
@@
 		(dnp no)
 		(fields_autoplaced yes)
-		(property "Reference" "D3"
+		(property "Reference" "D8"
 			(at 82.55 72.39 90)
 			(show_name no)
@@
 			(project "MIKA"
 				(path "/66ea9e27-3ca5-4edd-a0db-1f3995e73e78/c2d6fcaf-19aa-4c33-838f-5e0ce95c1959/7dc4223e-0f41-465d-891f-db8b5b137845"
-					(reference "D3")
+					(reference "D8")
 					(unit 1)
 				)
@@
 		(in_pos_files yes)
 		(dnp no)
-		(property "Reference" "C?"
+		(property "Reference" "C38"
 			(at 27.94 71.12 0)
 			(show_name no)
@@
 			)
 		)
-		(property "Value" "4.7nF"
-			(at 25.4 76.2 0)
+		(property "Value" "4.7n"
+			(at 26.67 76.2 0)
 			(show_name no)
 			(do_not_autoplace no)
@@
 			(project "MIKA"
 				(path "/66ea9e27-3ca5-4edd-a0db-1f3995e73e78/c2d6fcaf-19aa-4c33-838f-5e0ce95c1959/7dc4223e-0f41-465d-891f-db8b5b137845"
-					(reference "C?")
+					(reference "C38")
 					(unit 1)
 				)
@@
 		(in_pos_files yes)
 		(dnp no)
-		(property "Reference" "R?"
+		(property "Reference" "R22"
 			(at 21.59 74.93 90)
 			(show_name no)
@@
 			(project "MIKA"
 				(path "/66ea9e27-3ca5-4edd-a0db-1f3995e73e78/c2d6fcaf-19aa-4c33-838f-5e0ce95c1959/7dc4223e-0f41-465d-891f-db8b5b137845"
-					(reference "R?")
+					(reference "R22")
 					(unit 1)
 				)
@@
 		(dnp no)
 		(fields_autoplaced yes)
-		(property "Reference" "J1"
+		(property "Reference" "J12"
 			(at 35.56 22.86 0)
 			(show_name no)
@@
 			(project "MIKA"
 				(path "/66ea9e27-3ca5-4edd-a0db-1f3995e73e78/c2d6fcaf-19aa-4c33-838f-5e0ce95c1959/7dc4223e-0f41-465d-891f-db8b5b137845"
-					(reference "J1")
+					(reference "J12")
 					(unit 1)
 				)
@@
 		(in_pos_files yes)
 		(dnp no)
-		(property "Reference" "D1"
+		(property "Reference" "D7"
 			(at 59.69 24.765 0)
 			(show_name no)
@@
 			(project "MIKA"
 				(path "/66ea9e27-3ca5-4edd-a0db-1f3995e73e78/c2d6fcaf-19aa-4c33-838f-5e0ce95c1959/7dc4223e-0f41-465d-891f-db8b5b137845"
-					(reference "D1")
+					(reference "D7")
 					(unit 1)
 				)
@@
 		(in_pos_files yes)
 		(dnp no)
-		(property "Reference" "C1"
+		(property "Reference" "C39"
 			(at 64.3128 37.9984 0)
 			(show_name no)
@@
 			(project "MIKA"
 				(path "/66ea9e27-3ca5-4edd-a0db-1f3995e73e78/c2d6fcaf-19aa-4c33-838f-5e0ce95c1959/7dc4223e-0f41-465d-891f-db8b5b137845"
-					(reference "C1")
-					(unit 1)
-				)
+					(reference "C39")
+					(unit 1)
+				)

Commit message: bahasdf;ladjsfhadf boooooooooooshksa
Parts:
- removed C38: 4.7n, symbol Device:C
- removed R22: 1M, symbol Device:R
- added C39: 4.7n, symbol Device:C
- added C40: 1u, Capacitor_SMD:C_0805_2012Metric, symbol Device:C
- added C41: 0.1u, Capacitor_SMD:C_0805_2012Metric, symbol Device:C
- added C42: 2.2n, Capacitor_SMD:C_0805_2012Metric, symbol Device:C
- added C43: 1n, Capacitor_SMD:C_0805_2012Metric, symbol Device:C
- added D18: LED, LED_SMD:LED_0603_1608Metric, symbol Device:LED
- added IC3: TPS259480AYWPR, TPS259480AYWPR, symbol TPS259480AYWPR:TPS259480AYWPR
- added JP6: SolderJumper_2_Open, symbol Jumper:SolderJumper_2_Open
- added R41: 1M, symbol Device:R
- added R42: 390k, symbol Device:R
- added R43: 100k, symbol Device:R
- added R46: 2.2k, Resistor_SMD:R_0603_1608Metric_Pad0.98x0.95mm_HandSolder, symbol Device:R
- added R47: 820, symbol Device:R
- renumbered C39 to C44, D8 to D17, D7 to D19, J12 to J13, R23 to R44, R24 to R45
Connections:
- net GND: now also C39.2, C40.1, C41.1, C42.1, C43.1, IC3.8 (GND), R41.2, R43.2, R47.2
- net USB_5V: now also IC3.11 (VOUT_2), IC3.6 (VOUT_1)
- net at J13.S1 (SHIELD), J13.S2 (Shield), J13.S3 (Shield)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: now also C39.1, R41.1
- net VBUS_IN renamed UVLO
- net UVLO: now also C40.2, C41.2, D18.2 (A), IC3.1 (EN/UVLO), IC3.12 (VIN_2), IC3.5 (VIN_1), JP6.1 (A), R42.1; no longer D19.2 (A)
- new net: IC3.9 (ILM), R47.1
- new net: D19.2 (A), JP6.2 (B)
- new net: C42.2, IC3.10 (ITIMER)
- new net: D18.1 (K), R46.1
- new net: C43.2, IC3.7 (DVDT)
- new net FLT: IC3.4 (~{FLT}), R46.2
- new net OVLO: IC3.2 (OVLO), R42.2, R43.1
- no-connect marks 2 -> 3
Other:
- note added: "Ideal Diode IC"
- moved on the sheet: C44, D17, D19, J13, R44, R45
