File: Hardware/MIKA/ethernet.kicad_sch (KiCad schematic)
At the start: 6 parts

Commit message: ugahhghh might be layout time im a lil excited lwk
Parts:
- C46: renamed from C?; value 4.7nF -> 4.7n
- gave numbers to parts that had none: 5
Connections:
- no-connect marks 0 -> 2
Changed lines of the file:
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@@
 		(color 0 0 0 0)
+	)
+	(no_connect
+		(at 109.22 44.45)
+	)
+	(no_connect
+		(at 109.22 52.07)
 	)
 	(bus_entry
@@
 		(in_pos_files yes)
 		(dnp no)
-		(property "Reference" "R?"
+		(property "Reference" "R32"
 			(at 163.83 39.37 90)
 			(show_name no)
@@
 			(project "MIKA"
 				(path "/66ea9e27-3ca5-4edd-a0db-1f3995e73e78/c2d6fcaf-19aa-4c33-838f-5e0ce95c1959/735344d6-c3ef-403c-9e8c-4704de9e492d"
-					(reference "R?")
+					(reference "R32")
 					(unit 1)
 				)
@@
 		(in_pos_files yes)
 		(dnp no)
-		(property "Reference" "R?"
+		(property "Reference" "R31"
 			(at 138.43 67.31 90)
 			(show_name no)
@@
 			(project "MIKA"
 				(path "/66ea9e27-3ca5-4edd-a0db-1f3995e73e78/c2d6fcaf-19aa-4c33-838f-5e0ce95c1959/735344d6-c3ef-403c-9e8c-4704de9e492d"
-					(reference "R?")
+					(reference "R31")
 					(unit 1)
 				)
@@
 		(in_pos_files yes)
 		(dnp no)
-		(property "Reference" "R?"
+		(property "Reference" "R33"
 			(at 163.83 49.53 90)
 			(show_name no)
@@
 			(project "MIKA"
 				(path "/66ea9e27-3ca5-4edd-a0db-1f3995e73e78/c2d6fcaf-19aa-4c33-838f-5e0ce95c1959/735344d6-c3ef-403c-9e8c-4704de9e492d"
-					(reference "R?")
+					(reference "R33")
 					(unit 1)
 				)
@@
 		(dnp no)
 		(fields_autoplaced yes)
-		(property "Reference" "J?"
+		(property "Reference" "J15"
 			(at 130.81 35.56 0)
 			(show_name no)
@@
 			(project "MIKA"
 				(path "/66ea9e27-3ca5-4edd-a0db-1f3995e73e78/c2d6fcaf-19aa-4c33-838f-5e0ce95c1959/735344d6-c3ef-403c-9e8c-4704de9e492d"
-					(reference "J?")
+					(reference "J15")
 					(unit 1)
 				)
@@
 		(in_pos_files yes)
 		(dnp no)
-		(property "Reference" "C?"
+		(property "Reference" "C46"
 			(at 143.51 63.5 0)
 			(show_name no)
@@
 			)
 		)
-		(property "Value" "4.7nF"
+		(property "Value" "4.7n"
 			(at 143.51 68.58 0)
 			(show_name no)
@@
 			(project "MIKA"
 				(path "/66ea9e27-3ca5-4edd-a0db-1f3995e73e78/c2d6fcaf-19aa-4c33-838f-5e0ce95c1959/735344d6-c3ef-403c-9e8c-4704de9e492d"
-					(reference "C?")
+					(reference "C46")
 					(unit 1)
 				)
@@
 		(dnp no)
 		(fields_autoplaced yes)
-		(property "Reference" "U?"
+		(property "Reference" "U13"
 			(at 54.61 36.83 0)
 			(show_name no)
@@
 			(project "MIKA"
 				(path "/66ea9e27-3ca5-4edd-a0db-1f3995e73e78/c2d6fcaf-19aa-4c33-838f-5e0ce95c1959/735344d6-c3ef-403c-9e8c-4704de9e492d"
-					(reference "U?")
+					(reference "U13")
 					(unit 1)
 				)

Commit message: bahasdf;ladjsfhadf boooooooooooshksa
Parts:
- renumbered C46 to C51, J15 to J16, R31 to R54, R32 to R55, R33 to R56, U13 to U11
Changed lines of the file:
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@@
 		(in_pos_files yes)
 		(dnp no)
-		(property "Reference" "R32"
+		(property "Reference" "R55"
 			(at 163.83 39.37 90)
 			(show_name no)
@@
 			(project "MIKA"
 				(path "/66ea9e27-3ca5-4edd-a0db-1f3995e73e78/c2d6fcaf-19aa-4c33-838f-5e0ce95c1959/735344d6-c3ef-403c-9e8c-4704de9e492d"
-					(reference "R32")
+					(reference "R55")
 					(unit 1)
 				)
@@
 		(in_pos_files yes)
 		(dnp no)
-		(property "Reference" "R31"
+		(property "Reference" "R54"
 			(at 138.43 67.31 90)
 			(show_name no)
@@
 			(project "MIKA"
 				(path "/66ea9e27-3ca5-4edd-a0db-1f3995e73e78/c2d6fcaf-19aa-4c33-838f-5e0ce95c1959/735344d6-c3ef-403c-9e8c-4704de9e492d"
-					(reference "R31")
+					(reference "R54")
 					(unit 1)
 				)
@@
 		(in_pos_files yes)
 		(dnp no)
-		(property "Reference" "R33"
+		(property "Reference" "R56"
 			(at 163.83 49.53 90)
 			(show_name no)
@@
 			(project "MIKA"
 				(path "/66ea9e27-3ca5-4edd-a0db-1f3995e73e78/c2d6fcaf-19aa-4c33-838f-5e0ce95c1959/735344d6-c3ef-403c-9e8c-4704de9e492d"
-					(reference "R33")
+					(reference "R56")
 					(unit 1)
 				)
@@
 		(dnp no)
 		(fields_autoplaced yes)
-		(property "Reference" "J15"
+		(property "Reference" "J16"
 			(at 130.81 35.56 0)
 			(show_name no)
@@
 			(project "MIKA"
 				(path "/66ea9e27-3ca5-4edd-a0db-1f3995e73e78/c2d6fcaf-19aa-4c33-838f-5e0ce95c1959/735344d6-c3ef-403c-9e8c-4704de9e492d"
-					(reference "J15")
+					(reference "J16")
 					(unit 1)
 				)
@@
 		(in_pos_files yes)
 		(dnp no)
-		(property "Reference" "C46"
+		(property "Reference" "C51"
 			(at 143.51 63.5 0)
 			(show_name no)
@@
 			(project "MIKA"
 				(path "/66ea9e27-3ca5-4edd-a0db-1f3995e73e78/c2d6fcaf-19aa-4c33-838f-5e0ce95c1959/735344d6-c3ef-403c-9e8c-4704de9e492d"
-					(reference "C46")
+					(reference "C51")
 					(unit 1)
 				)
@@
 		(dnp no)
 		(fields_autoplaced yes)
-		(property "Reference" "U13"
+		(property "Reference" "U11"
 			(at 54.61 36.83 0)
 			(show_name no)
@@
 			(project "MIKA"
 				(path "/66ea9e27-3ca5-4edd-a0db-1f3995e73e78/c2d6fcaf-19aa-4c33-838f-5e0ce95c1959/735344d6-c3ef-403c-9e8c-4704de9e492d"
-					(reference "U13")
-					(unit 1)
-				)
+					(reference "U11")
+					(unit 1)
+				)
