File: Hardware/MIKA/hdmi_out.kicad_sch (KiCad schematic)
At the start: 14 parts

Commit message: ugahhghh might be layout time im a lil excited lwk
Parts:
- removed C?: 100nF, symbol Device:C
- added C?: 0.1u, symbol Device:C
- C41: renamed from C?; value 47uF -> 47u
- C42: renamed from C?; value 4.7nF -> 4.7n
- gave numbers to parts that had none: 11
Connections:
- net +5V: now also C?.2
- net GND: now also C?.1
Changed lines of the file:
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@@
 	)
 	(junction
-		(at 87.63 58.42)
+		(at 52.07 40.64)
 		(diameter 0)
 		(color 0 0 0 0)
 	)
 	(junction
-		(at 175.26 111.76)
+		(at 87.63 58.42)
 		(diameter 0)
 		(color 0 0 0 0)
 	)
 	(junction
-		(at 162.56 100.33)
+		(at 175.26 111.76)
 		(diameter 0)
 		(color 0 0 0 0)
 	)
 	(junction
-		(at 87.63 40.64)
+		(at 162.56 100.33)
 		(diameter 0)
 		(color 0 0 0 0)
 	)
 	(junction
-		(at 52.07 40.64)
+		(at 87.63 40.64)
 		(diameter 0)
 		(color 0 0 0 0)
@@
 	(wire
 		(pts
-			(xy 52.07 40.64) (xy 54.61 40.64)
+			(xy 137.16 54.61) (xy 153.67 54.61)
 		)
 		(stroke
@@
 	(wire
 		(pts
-			(xy 137.16 54.61) (xy 153.67 54.61)
+			(xy 163.83 34.29) (xy 163.83 44.45)
 		)
 		(stroke
@@
 		)
 	)
-	(wire
+	(bus
 		(pts
-			(xy 163.83 34.29) (xy 163.83 44.45)
+			(xy 46.99 81.28) (xy 46.99 157.48)
 		)
 		(stroke
@@
 		)
 	)
-	(bus
+	(wire
 		(pts
-			(xy 46.99 81.28) (xy 46.99 157.48)
+			(xy 52.07 40.64) (xy 54.61 40.64)
 		)
 		(stroke
@@
 		(in_pos_files yes)
 		(dnp no)
-		(property "Reference" "R?"
+		(property "Reference" "R25"
 			(at 83.82 49.53 0)
 			(show_name no)
@@
 			(project "MIKA"
 				(path "/66ea9e27-3ca5-4edd-a0db-1f3995e73e78/c2d6fcaf-19aa-4c33-838f-5e0ce95c1959/be6c36fa-6fd6-406f-a5ea-75fa261ef4c4"
-					(reference "R?")
+					(reference "R25")
+					(unit 1)
+				)
+			)
+		)
+	)
+	(symbol
+		(lib_id "Device:C")
+		(at 52.07 44.45 0)
+		(mirror x)
+		(unit 1)
+		(body_style 1)
+		(exclude_from_sim no)
+		(in_bom yes)
+		(on_board yes)
+		(in_pos_files yes)
+		(dnp no)
+		(property "Reference" "C?"
+			(at 50.165 41.91 0)
+			(show_name no)
+			(do_not_autoplace no)
+			(effects
+				(font
+					(size 1.27 1.27)
+				)
+			)
+		)
+		(property "Value" "0.1u"
+			(at 49.53 46.99 0)
+			(show_name no)
+			(do_not_autoplace no)
+			(effects
+				(font
+					(size 1.27 1.27)
+				)
+			)
+		)
+		(property "Footprint" ""
+			(at 53.0352 40.64 0)
+			(hide yes)
+			(show_name no)
+			(do_not_autoplace no)
+			(effects
+				(font
+					(size 1.27 1.27)
+				)
+			)
+		)
+		(property "Datasheet" ""
+			(at 52.07 44.45 0)
+			(hide yes)
+			(show_name no)
+			(do_not_autoplace no)
+			(effects
+				(font
+					(size 1.27 1.27)
+				)
+			)
+		)
+		(property "Description" "Unpolarized capacitor"
+			(at 52.07 44.45 0)
+			(hide yes)
+			(show_name no)
+			(do_not_autoplace no)
+			(effects
+				(font
+					(size 1.27 1.27)
+				)
+			)
+		)
+		(pin "1"
+		)
+		(pin "2"
+		)
+		(instances
+			(project "MIKA"
+				(path "/66ea9e27-3ca5-4edd-a0db-1f3995e73e78/c2d6fcaf-19aa-4c33-838f-5e0ce95c1959/be6c36fa-6fd6-406f-a5ea-75fa261ef4c4"
+					(reference "C?")
 					(unit 1)
 				)
@@
 		(dnp no)
 		(fields_autoplaced yes)
-		(property "Reference" "U?"
+		(property "Reference" "U8"
 			(at 74.93 144.78 0)
 			(show_name no)
@@
 			(project "MIKA"
 				(path "/66ea9e27-3ca5-4edd-a0db-1f3995e73e78/c2d6fcaf-19aa-4c33-838f-5e0ce95c1959/be6c36fa-6fd6-406f-a5ea-75fa261ef4c4"
-					(reference "U?")
+					(reference "U8")
 					(unit 1)
 				)
@@
 		(in_pos_files yes)
 		(dnp no)
-		(property "Reference" "U?"
+		(property "Reference" "U9"
 			(at 147.32 36.2584 0)
 			(show_name no)
@@
 			(project "MIKA"
 				(path "/66ea9e27-3ca5-4edd-a0db-1f3995e73e78/c2d6fcaf-19aa-4c33-838f-5e0ce95c1959/be6c36fa-6fd6-406f-a5ea-75fa261ef4c4"
-					(reference "U?")
+					(reference "U9")
 					(unit 1)
 				)
@@
 		(in_pos_files yes)
 		(dnp no)
-		(property "Reference" "D?"
+		(property "Reference" "D9"
 			(at 93.98 34.29 0)
 			(show_name no)
@@
 			(project "MIKA"
 				(path "/66ea9e27-3ca5-4edd-a0db-1f3995e73e78/c2d6fcaf-19aa-4c33-838f-5e0ce95c1959/be6c36fa-6fd6-406f-a5ea-75fa261ef4c4"
-					(reference "D?")
+					(reference "D9")
 					(unit 1)
 				)
@@
 		(dnp no)
 		(fields_autoplaced yes)
-		(property "Reference" "IC?"
+		(property "Reference" "IC2"
 			(at 71.12 29.21 0)
 			(show_name no)
@@
 			(project "MIKA"
 				(path "/66ea9e27-3ca5-4edd-a0db-1f3995e73e78/c2d6fcaf-19aa-4c33-838f-5e0ce95c1959/be6c36fa-6fd6-406f-a5ea-75fa261ef4c4"
-					(reference "IC?")
+					(reference "IC2")
 					(unit 1)
 				)
@@
 		(in_pos_files yes)
 		(dnp no)
-		(property "Reference" "R?"
+		(property "Reference" "R26"
 			(at 101.6 34.29 90)
 			(show_name no)
@@
 			(project "MIKA"
 				(path "/66ea9e27-3ca5-4edd-a0db-1f3995e73e78/c2d6fcaf-19aa-4c33-838f-5e0ce95c1959/be6c36fa-6fd6-406f-a5ea-75fa261ef4c4"
-					(reference "R?")
+					(reference "R26")
 					(unit 1)
 				)
@@
 		(in_pos_files yes)
 		(dnp no)
-		(property "Reference" "R?"
+		(property "Reference" "R27"
 			(at 173.99 107.95 90)
 			(show_name no)
@@
 			(project "MIKA"
 				(path "/66ea9e27-3ca5-4edd-a0db-1f3995e73e78/c2d6fcaf-19aa-4c33-838f-5e0ce95c1959/be6c36fa-6fd6-406f-a5ea-75fa261ef4c4"
-					(reference "R?")
+					(reference "R27")
 					(unit 1)
 				)
@@
 		(in_pos_files yes)
 		(dnp no)
-		(property "Reference" "FB?"
+		(property "Reference" "FB1"
 			(at 153.67 27.94 90)
 			(show_name no)
@@
 			(project "MIKA"
 				(path "/66ea9e27-3ca5-4edd-a0db-1f3995e73e78/c2d6fcaf-19aa-4c33-838f-5e0ce95c1959/be6c36fa-6fd6-406f-a5ea-75fa261ef4c4"
-					(reference "FB?")
+					(reference "FB1")
 					(unit 1)
 				)
@@
 		(dnp no)
 		(fields_autoplaced yes)
-		(property "Reference" "U?"
+		(property "Reference" "U6"
 			(at 74.93 73.66 0)
 			(show_name no)
@@
 			(project "MIKA"
 				(path "/66ea9e27-3ca5-4edd-a0db-1f3995e73e78/c2d6fcaf-19aa-4c33-838f-5e0ce95c1959/be6c36fa-6fd6-406f-a5ea-75fa261ef4c4"
-					(reference "U?")
+					(reference "U6")
 					(unit 1)
 				)
@@
 		(in_pos_files yes)
 		(dnp no)
-		(property "Reference" "C?"
-			(at 158.75 34.29 0)
+		(property "Reference" "C41"
+			(at 157.48 34.29 0)
 			(show_name no)
 			(do_not_autoplace no)
@@
 			)
 		)
-		(property "Value" "47uF"
+		(property "Value" "47u"
 			(at 157.48 39.37 0)
 			(show_name no)
@@
 			(project "MIKA"
 				(path "/66ea9e27-3ca5-4edd-a0db-1f3995e73e78/c2d6fcaf-19aa-4c33-838f-5e0ce95c1959/be6c36fa-6fd6-406f-a5ea-75fa261ef4c4"
-					(reference "C?")
+					(reference "C41")
 					(unit 1)
 				)
@@
 		(dnp no)
 		(fields_autoplaced yes)
-		(property "Reference" "U?"
+		(property "Reference" "U7"
 			(at 74.93 109.22 0)
 			(show_name no)
@@
 			(project "MIKA"
 				(path "/66ea9e27-3ca5-4edd-a0db-1f3995e73e78/c2d6fcaf-19aa-4c33-838f-5e0ce95c1959/be6c36fa-6fd6-406f-a5ea-75fa261ef4c4"
-					(reference "U?")
-					(unit 1)
-				)
-			)
-		)
-	)
-	(symbol
-		(lib_id "Device:C")
-		(at 52.07 44.45 0)
-		(unit 1)
-		(body_style 1)
-		(exclude_from_sim no)
-		(in_bom yes)
-		(on_board yes)
-		(in_pos_files yes)
-		(dnp no)
-		(property "Reference" "C?"
-			(at 49.53 41.91 0)
-			(show_name no)
-			(do_not_autoplace no)
-			(effects
-				(font
-					(size 1.27 1.27)
-				)
-				(justify left)
-			)
-		)
-		(property "Value" "100nF"
-			(at 45.72 46.99 0)
-			(show_name no)
-			(do_not_autoplace no)
-			(effects
-				(font
-					(size 1.27 1.27)
-				)
-				(justify left)
-			)
-		)
-		(property "Footprint" ""
-			(at 53.0352 48.26 0)
-			(hide yes)
-			(show_name no)
-			(do_not_autoplace no)
-			(effects
-				(font
-					(size 1.27 1.27)
-				)
-			)
-		)
-		(property "Datasheet" ""
-			(at 52.07 44.45 0)
-			(hide yes)
-			(show_name no)
-			(do_not_autoplace no)
-			(effects
-				(font
-					(size 1.27 1.27)
-				)
-			)
-		)
-		(property "Description" "Unpolarized capacitor"
-			(at 52.07 44.45 0)
-			(hide yes)
-			(show_name no)
-			(do_not_autoplace no)
-			(effects
-				(font
-					(size 1.27 1.27)
-				)
-			)
-		)
-		(pin "1"
-		)
-		(pin "2"
-		)
-		(instances
-			(project "MIKA"
-				(path "/66ea9e27-3ca5-4edd-a0db-1f3995e73e78/c2d6fcaf-19aa-4c33-838f-5e0ce95c1959/be6c36fa-6fd6-406f-a5ea-75fa261ef4c4"
-					(reference "C?")
+					(reference "U7")
 					(unit 1)
 				)
@@
 		(dnp no)
 		(fields_autoplaced yes)
-		(property "Reference" "J?"
+		(property "Reference" "J13"
 			(at 175.26 71.1199 0)
 			(show_name no)
@@
 			(project "MIKA"
 				(path "/66ea9e27-3ca5-4edd-a0db-1f3995e73e78/c2d6fcaf-19aa-4c33-838f-5e0ce95c1959/be6c36fa-6fd6-406f-a5ea-75fa261ef4c4"
-					(reference "J?")
+					(reference "J13")
 					(unit 1)
 				)
@@
 		(in_pos_files yes)
 		(dnp no)
-		(property "Reference" "C?"
+		(property "Reference" "C42"
 			(at 179.07 104.14 0)
 			(show_name no)
@@
 			)
 		)
-		(property "Value" "4.7nF"
+		(property "Value" "4.7n"
 			(at 179.07 109.22 0)
 			(show_name no)
@@
 			(project "MIKA"
 				(path "/66ea9e27-3ca5-4edd-a0db-1f3995e73e78/c2d6fcaf-19aa-4c33-838f-5e0ce95c1959/be6c36fa-6fd6-406f-a5ea-75fa261ef4c4"
-					(reference "C?")
+					(reference "C42")
 					(unit 1)
 				)

Commit message: bahasdf;ladjsfhadf boooooooooooshksa
Parts:
- gave numbers to parts that had none: 1
- renumbered C41 to C46, C42 to C47, D9 to D20, IC2 to IC4, J13 to J14, R25 to R48, R26 to R49, R27 to R50, U6 to U4, U7 to U5, U8 to U6, U9 to U7
Other:
- note added: "add desmos math 4 ravi"
Changed lines of the file:
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@@
 		)
 	)
+	(text "add desmos math 4 ravi"
+		(exclude_from_sim no)
+		(at 84.455 62.23 0)
+		(effects
+			(font
+				(size 1.27 1.27)
+			)
+		)
+	)
 	(text "Ilim: ~500mA"
 		(exclude_from_sim no)
@@
 		(in_pos_files yes)
 		(dnp no)
-		(property "Reference" "R25"
-			(at 83.82 49.53 0)
+		(property "Reference" "R48"
+			(at 83.185 48.26 0)
 			(show_name no)
 			(do_not_autoplace no)
@@
 			(project "MIKA"
 				(path "/66ea9e27-3ca5-4edd-a0db-1f3995e73e78/c2d6fcaf-19aa-4c33-838f-5e0ce95c1959/be6c36fa-6fd6-406f-a5ea-75fa261ef4c4"
-					(reference "R25")
+					(reference "R48")
 					(unit 1)
 				)
@@
 		(in_pos_files yes)
 		(dnp no)
-		(property "Reference" "C?"
+		(property "Reference" "C45"
 			(at 50.165 41.91 0)
 			(show_name no)
@@
 			(project "MIKA"
 				(path "/66ea9e27-3ca5-4edd-a0db-1f3995e73e78/c2d6fcaf-19aa-4c33-838f-5e0ce95c1959/be6c36fa-6fd6-406f-a5ea-75fa261ef4c4"
-					(reference "C?")
+					(reference "C45")
 					(unit 1)
 				)
@@
 		(dnp no)
 		(fields_autoplaced yes)
-		(property "Reference" "U8"
+		(property "Reference" "U6"
 			(at 74.93 144.78 0)
 			(show_name no)
@@
 			(project "MIKA"
 				(path "/66ea9e27-3ca5-4edd-a0db-1f3995e73e78/c2d6fcaf-19aa-4c33-838f-5e0ce95c1959/be6c36fa-6fd6-406f-a5ea-75fa261ef4c4"
-					(reference "U8")
+					(reference "U6")
 					(unit 1)
 				)
@@
 		(in_pos_files yes)
 		(dnp no)
-		(property "Reference" "U9"
+		(property "Reference" "U7"
 			(at 147.32 36.2584 0)
 			(show_name no)
@@
 			(project "MIKA"
 				(path "/66ea9e27-3ca5-4edd-a0db-1f3995e73e78/c2d6fcaf-19aa-4c33-838f-5e0ce95c1959/be6c36fa-6fd6-406f-a5ea-75fa261ef4c4"
-					(reference "U9")
+					(reference "U7")
 					(unit 1)
 				)
@@
 		(in_pos_files yes)
 		(dnp no)
-		(property "Reference" "D9"
+		(property "Reference" "D20"
 			(at 93.98 34.29 0)
 			(show_name no)
@@
 			(project "MIKA"
 				(path "/66ea9e27-3ca5-4edd-a0db-1f3995e73e78/c2d6fcaf-19aa-4c33-838f-5e0ce95c1959/be6c36fa-6fd6-406f-a5ea-75fa261ef4c4"
-					(reference "D9")
+					(reference "D20")
 					(unit 1)
 				)
@@
 		(dnp no)
 		(fields_autoplaced yes)
-		(property "Reference" "IC2"
+		(property "Reference" "IC4"
 			(at 71.12 29.21 0)
 			(show_name no)
@@
 			(project "MIKA"
 				(path "/66ea9e27-3ca5-4edd-a0db-1f3995e73e78/c2d6fcaf-19aa-4c33-838f-5e0ce95c1959/be6c36fa-6fd6-406f-a5ea-75fa261ef4c4"
-					(reference "IC2")
+					(reference "IC4")
 					(unit 1)
 				)
@@
 		(in_pos_files yes)
 		(dnp no)
-		(property "Reference" "R26"
+		(property "Reference" "R49"
 			(at 101.6 34.29 90)
 			(show_name no)
@@
 			(project "MIKA"
 				(path "/66ea9e27-3ca5-4edd-a0db-1f3995e73e78/c2d6fcaf-19aa-4c33-838f-5e0ce95c1959/be6c36fa-6fd6-406f-a5ea-75fa261ef4c4"
-					(reference "R26")
+					(reference "R49")
 					(unit 1)
 				)
@@
 		(in_pos_files yes)
 		(dnp no)
-		(property "Reference" "R27"
+		(property "Reference" "R50"
 			(at 173.99 107.95 90)
 			(show_name no)
@@
 			(project "MIKA"
 				(path "/66ea9e27-3ca5-4edd-a0db-1f3995e73e78/c2d6fcaf-19aa-4c33-838f-5e0ce95c1959/be6c36fa-6fd6-406f-a5ea-75fa261ef4c4"
-					(reference "R27")
+					(reference "R50")
 					(unit 1)
 				)
@@
 		(dnp no)
 		(fields_autoplaced yes)
-		(property "Reference" "U6"
+		(property "Reference" "U4"
 			(at 74.93 73.66 0)
 			(show_name no)
@@
 			(project "MIKA"
 				(path "/66ea9e27-3ca5-4edd-a0db-1f3995e73e78/c2d6fcaf-19aa-4c33-838f-5e0ce95c1959/be6c36fa-6fd6-406f-a5ea-75fa261ef4c4"
-					(reference "U6")
+					(reference "U4")
 					(unit 1)
 				)
@@
 		(in_pos_files yes)
 		(dnp no)
-		(property "Reference" "C41"
+		(property "Reference" "C46"
 			(at 157.48 34.29 0)
 			(show_name no)
@@
 			(project "MIKA"
 				(path "/66ea9e27-3ca5-4edd-a0db-1f3995e73e78/c2d6fcaf-19aa-4c33-838f-5e0ce95c1959/be6c36fa-6fd6-406f-a5ea-75fa261ef4c4"
-					(reference "C41")
+					(reference "C46")
 					(unit 1)
 				)
@@
 		(dnp no)
 		(fields_autoplaced yes)
-		(property "Reference" "U7"
+		(property "Reference" "U5"
 			(at 74.93 109.22 0)
 			(show_name no)
@@
 			(project "MIKA"
 				(path "/66ea9e27-3ca5-4edd-a0db-1f3995e73e78/c2d6fcaf-19aa-4c33-838f-5e0ce95c1959/be6c36fa-6fd6-406f-a5ea-75fa261ef4c4"
-					(reference "U7")
+					(reference "U5")
 					(unit 1)
 				)
@@
 		(dnp no)
 		(fields_autoplaced yes)
-		(property "Reference" "J13"
+		(property "Reference" "J14"
 			(at 175.26 71.1199 0)
 			(show_name no)
@@
 			(project "MIKA"
 				(path "/66ea9e27-3ca5-4edd-a0db-1f3995e73e78/c2d6fcaf-19aa-4c33-838f-5e0ce95c1959/be6c36fa-6fd6-406f-a5ea-75fa261ef4c4"
-					(reference "J13")
+					(reference "J14")
 					(unit 1)
 				)
@@
 		(in_pos_files yes)
 		(dnp no)
-		(property "Reference" "C42"
+		(property "Reference" "C47"
 			(at 179.07 104.14 0)
 			(show_name no)
@@
 			(project "MIKA"
 				(path "/66ea9e27-3ca5-4edd-a0db-1f3995e73e78/c2d6fcaf-19aa-4c33-838f-5e0ce95c1959/be6c36fa-6fd6-406f-a5ea-75fa261ef4c4"
-					(reference "C42")
+					(reference "C47")
 					(unit 1)
 				)
