File: Hardware/MIKA/high_speed.kicad_sch (KiCad schematic)
At the start: 1 part

Commit message: ugahhghh might be layout time im a lil excited lwk
Parts:
- gave numbers to parts that had none: 1
Changed lines of the file:
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@@
 		(dnp no)
 		(fields_autoplaced yes)
-		(property "Reference" "Module?"
+		(property "Reference" "Module1"
 			(at 86.36 27.94 0)
 			(show_name no)
@@
 			(project "MIKA"
 				(path "/66ea9e27-3ca5-4edd-a0db-1f3995e73e78/c2d6fcaf-19aa-4c33-838f-5e0ce95c1959"
-					(reference "Module?")
+					(reference "Module1")
 					(unit 2)
 				)

Commit message: bahasdf;ladjsfhadf boooooooooooshksa
Connections:
- net USB_DN renamed USB_D-
- net USB_DP renamed USB_D+
Changed lines of the file:
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@@
+	)
+	(bus_entry
+		(at 39.37 147.32)
+		(size 2.54 2.54)
+		(stroke
+			(width 0)
+			(type default)
+		)
 	)
 	(bus_entry
@@
 		)
 	)
-	(label "USB_DP"
+	(label "USB_D+"
+		(at 125.73 45.72 180)
+		(effects
+			(font
+				(size 1.27 1.27)
+			)
+			(justify right bottom)
+		)
+	)
+	(label "USB_D+"
 		(at 207.01 59.69 0)
 		(effects
@@
 			)
 			(justify left bottom)
-		)
-	)
-	(label "USB_DN"
-		(at 125.73 43.18 180)
-		(effects
-			(font
-				(size 1.27 1.27)
-			)
-			(justify right bottom)
 		)
 	)
@@
 		)
 	)
-	(label "USB_DN"
+	(label "USB_D-"
 		(at 207.01 62.23 0)
 		(effects
@@
 		)
 	)
-	(label "USB_DP"
-		(at 125.73 45.72 180)
-		(effects
-			(font
-				(size 1.27 1.27)
-			)
-			(justify right bottom)
-		)
-	)
 	(label "HDMI0_D1_N"
 		(at 41.91 137.16 0)
@@
 			)
 			(justify left bottom)
+		)
+	)
+	(label "USB_D-"
+		(at 125.73 43.18 180)
+		(effects
+			(font
+				(size 1.27 1.27)
+			)
+			(justify right bottom)
 		)
 	)
@@
 		)
 		(property "Author" "Shuopu Wang"
-			(at 71.12 -81.28 0)
+			(at 0 0.635 0)
 			(hide yes)
 			(show_name no)
@@
 		)
 		(property "Date Modified" "9/5/2026"
-			(at 71.12 -81.28 0)
+			(at 0 0.635 0)
 			(hide yes)
 			(show_name no)
