File: Hardware/MIKA/usb_a_3.0.kicad_sch (KiCad schematic)
At the start: 13 parts

Commit message: ugahhghh might be layout time im a lil excited lwk
Parts:
- removed C?: 100n, symbol Device:C
- removed C?: 100nF, symbol Device:C
- added C? (x2): 0.1u, symbol Device:C
- C45: renamed from C?; value 4.7nF -> 4.7n
- gave numbers to parts that had none: 10
Connections:
- net +5V: now also C?.2
- net GND: now also C?.1, C?.1
- net at FB2.2, J14.1 (VBUS): now also C?.2

Commit message: bahasdf;ladjsfhadf boooooooooooshksa
Parts:
- gave numbers to parts that had none: 2
- renumbered C45 to C50, D10 to D21, IC3 to IC5, J14 to J15, R28 to R51, R29 to R52, R30 to R53, U12 to U10, U10 to U8, U11 to U9
Connections:
- net USB_HUB_D+ is gone; now on net USB3-0-D_P: U8.1 (D1+)
- net USB_HUB_D- is gone; now on net USB3-0-D_N: U8.2 (D1-)
- net USB_HUB_RX+ is gone; now on net USB3-0-RX_P: U8.4 (D2+)
- net USB_HUB_RX- is gone; now on net USB3-0-RX_N: U8.5 (D2-)
- net USB_HUB_TX+ is gone; now on net USB3-0-TX_P: U9.1 (D1+)
- net USB_HUB_TX- is gone; now on net USB3-0-TX_N: U9.2 (D1-)
Other:
- note added: "add desmos math 4 ravi"
Changed lines of the file:
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@@
+		)
+	)
+	(text "add desmos math 4 ravi"
+		(exclude_from_sim no)
+		(at 74.295 56.515 0)
+		(effects
+			(font
+				(size 1.27 1.27)
+			)
 		)
 	)
@@
 	(wire
 		(pts
+			(xy 66.04 106.68) (xy 80.01 106.68)
+		)
+		(stroke
+			(width 0)
+			(type default)
+		)
+	)
+	(wire
+		(pts
 			(xy 149.86 29.21) (xy 152.4 31.75)
 		)
@@
 	(wire
 		(pts
-			(xy 80.01 106.68) (xy 66.04 106.68)
-		)
-		(stroke
-			(width 0)
-			(type default)
-		)
-	)
-	(wire
-		(pts
 			(xy 152.4 31.75) (xy 152.4 41.91)
 		)
@@
 	(wire
 		(pts
+			(xy 66.04 111.76) (xy 80.01 111.76)
+		)
+		(stroke
+			(width 0)
+			(type default)
+		)
+	)
+	(wire
+		(pts
 			(xy 77.47 52.07) (xy 78.74 52.07)
 		)
@@
 		)
 	)
-	(wire
-		(pts
-			(xy 80.01 111.76) (xy 66.04 111.76)
-		)
-		(stroke
-			(width 0)
-			(type default)
-		)
-	)
 	(image
-		(at 87.63 45.72)
+		(at 88.265 45.72)
 		(scale 0.319188)
 		(data "iVBORw0KGgoAAAANSUhEUgAAAioAAAEtCAYAAAAm3UuWAAAABHNCSVQICAgIfAhkiAAAIABJREFU"
@@
 		)
 	)
-	(label "USB_HUB_D-"
-		(at 26.67 80.01 0)
-		(effects
-			(font
-				(size 1.27 1.27)
-				(thickness 0.1588)
-			)
-			(justify left bottom)
-		)
-	)
-	(label "USB_HUB_D+"
-		(at 26.67 74.93 0)
-		(effects
-			(font
-				(size 1.27 1.27)
-				(thickness 0.1588)
-			)
-			(justify left bottom)
-		)
-	)
 	(label "USB3-0-D_P"
 		(at 140.97 50.8 0)
@@
 		)
 	)
-	(label "USB_HUB_RX+"
-		(at 80.01 74.93 180)
-		(effects
-			(font
-				(size 1.27 1.27)
-				(thickness 0.1588)
-			)
-			(justify right bottom)
-		)
-	)
-	(label "USB_HUB_TX+"
+	(label "USB3-0-TX_P"
 		(at 80.01 106.68 180)
 		(effects
@@
 		)
 	)
-	(label "USB_HUB_RX-"
-		(at 80.01 80.01 180)
-		(effects
-			(font
-				(size 1.27 1.27)
-				(thickness 0.1588)
-			)
-			(justify right bottom)
-		)
-	)
 	(label "USB3-0-D_N"
 		(at 140.97 48.26 0)
@@
 		)
 	)
+	(label "USB3-0-D_P"
+		(at 26.67 74.93 0)
+		(effects
+			(font
+				(size 1.27 1.27)
+				(thickness 0.1588)
+			)
+			(justify left bottom)
+		)
+	)
+	(label "USB3-0-RX_N"
+		(at 80.01 80.01 180)
+		(effects
+			(font
+				(size 1.27 1.27)
+				(thickness 0.1588)
+			)
+			(justify right bottom)
+		)
+	)
+	(label "USB3-0-TX_N"
+		(at 80.01 111.76 180)
+		(effects
+			(font
+				(size 1.27 1.27)
+				(thickness 0.1588)
+			)
+			(justify right bottom)
+		)
+	)
 	(label "USB3-0-RX_N"
 		(at 140.97 55.88 0)
@@
 		)
 	)
+	(label "USB3-0-D_N"
+		(at 26.67 80.01 0)
+		(effects
+			(font
+				(size 1.27 1.27)
+				(thickness 0.1588)
+			)
+			(justify left bottom)
+		)
+	)
 	(label "USB3-0-TX_N"
 		(at 140.97 63.5 0)
@@
 		)
 	)
-	(label "USB_HUB_TX-"
-		(at 80.01 111.76 180)
+	(label "USB3-0-RX_P"
+		(at 80.01 74.93 180)
 		(effects
 			(font
@@
 		(dnp no)
 		(fields_autoplaced yes)
-		(property "Reference" "J14"
+		(property "Reference" "J15"
 			(at 167.64 34.29 0)
 			(show_name no)
@@
 			(project "MIKA"
 				(path "/66ea9e27-3ca5-4edd-a0db-1f3995e73e78/c2d6fcaf-19aa-4c33-838f-5e0ce95c1959/7a043766-a0c2-4407-9464-91c0fba921a3"
-					(reference "J14")
+					(reference "J15")
 					(unit 1)
 				)
@@
 		(dnp no)
 		(fields_autoplaced yes)
-		(property "Reference" "IC3"
+		(property "Reference" "IC5"
 			(at 60.96 22.86 0)
 			(show_name no)
@@
 			(project "MIKA"
 				(path "/66ea9e27-3ca5-4edd-a0db-1f3995e73e78/c2d6fcaf-19aa-4c33-838f-5e0ce95c1959/7a043766-a0c2-4407-9464-91c0fba921a3"
-					(reference "IC3")
+					(reference "IC5")
 					(unit 1)
 				)
@@
 		(in_pos_files yes)
 		(dnp no)
-		(property "Reference" "R28"
-			(at 73.66 43.18 0)
+		(property "Reference" "R51"
+			(at 73.025 41.91 0)
 			(show_name no)
 			(do_not_autoplace no)
@@
 			(project "MIKA"
 				(path "/66ea9e27-3ca5-4edd-a0db-1f3995e73e78/c2d6fcaf-19aa-4c33-838f-5e0ce95c1959/7a043766-a0c2-4407-9464-91c0fba921a3"
-					(reference "R28")
+					(reference "R51")
 					(unit 1)
 				)
@@
 		(in_pos_files yes)
 		(dnp no)
-		(property "Reference" "U11"
+		(property "Reference" "U9"
 			(at 53.34 96.52 0)
 			(show_name no)
@@
 			(project "MIKA"
 				(path "/66ea9e27-3ca5-4edd-a0db-1f3995e73e78/c2d6fcaf-19aa-4c33-838f-5e0ce95c1959/7a043766-a0c2-4407-9464-91c0fba921a3"
-					(reference "U11")
+					(reference "U9")
 					(unit 1)
 				)
@@
 		(in_pos_files yes)
 		(dnp no)
-		(property "Reference" "D10"
+		(property "Reference" "D21"
 			(at 83.82 27.94 0)
 			(show_name no)
@@
 			(project "MIKA"
 				(path "/66ea9e27-3ca5-4edd-a0db-1f3995e73e78/c2d6fcaf-19aa-4c33-838f-5e0ce95c1959/7a043766-a0c2-4407-9464-91c0fba921a3"
-					(reference "D10")
+					(reference "D21")
 					(unit 1)
 				)
@@
 		(in_pos_files yes)
 		(dnp no)
-		(property "Reference" "C?"
+		(property "Reference" "C49"
 			(at 147.955 31.75 0)
 			(show_name no)
@@
 			(project "MIKA"
 				(path "/66ea9e27-3ca5-4edd-a0db-1f3995e73e78/c2d6fcaf-19aa-4c33-838f-5e0ce95c1959/7a043766-a0c2-4407-9464-91c0fba921a3"
-					(reference "C?")
+					(reference "C49")
 					(unit 1)
 				)
@@
 		(in_pos_files yes)
 		(dnp no)
-		(property "Reference" "C?"
+		(property "Reference" "C48"
 			(at 40.64 36.195 0)
 			(show_name no)
@@
 			(project "MIKA"
 				(path "/66ea9e27-3ca5-4edd-a0db-1f3995e73e78/c2d6fcaf-19aa-4c33-838f-5e0ce95c1959/7a043766-a0c2-4407-9464-91c0fba921a3"
-					(reference "C?")
+					(reference "C48")
 					(unit 1)
 				)
@@
 		(in_pos_files yes)
 		(dnp no)
-		(property "Reference" "C45"
+		(property "Reference" "C50"
 			(at 176.53 76.2 0)
 			(show_name no)
@@
 			(project "MIKA"
 				(path "/66ea9e27-3ca5-4edd-a0db-1f3995e73e78/c2d6fcaf-19aa-4c33-838f-5e0ce95c1959/7a043766-a0c2-4407-9464-91c0fba921a3"
-					(reference "C45")
+					(reference "C50")
 					(unit 1)
 				)
@@
 		(in_pos_files yes)
 		(dnp no)
-		(property "Reference" "U12"
+		(property "Reference" "U10"
 			(at 138.43 33.7184 0)
 			(show_name no)
@@
 			(project "MIKA"
 				(path "/66ea9e27-3ca5-4edd-a0db-1f3995e73e78/c2d6fcaf-19aa-4c33-838f-5e0ce95c1959/7a043766-a0c2-4407-9464-91c0fba921a3"
-					(reference "U12")
+					(reference "U10")
 					(unit 1)
 				)
@@
 		(dnp no)
 		(fields_autoplaced yes)
-		(property "Reference" "U10"
+		(property "Reference" "U8"
 			(at 53.34 64.77 0)
 			(show_name no)
@@
 			(project "MIKA"
 				(path "/66ea9e27-3ca5-4edd-a0db-1f3995e73e78/c2d6fcaf-19aa-4c33-838f-5e0ce95c1959/7a043766-a0c2-4407-9464-91c0fba921a3"
-					(reference "U10")
+					(reference "U8")
 					(unit 1)
 				)
@@
 		(in_pos_files yes)
 		(dnp no)
-		(property "Reference" "R29"
+		(property "Reference" "R52"
 			(at 91.44 27.94 90)
 			(show_name no)
@@
 			(project "MIKA"
 				(path "/66ea9e27-3ca5-4edd-a0db-1f3995e73e78/c2d6fcaf-19aa-4c33-838f-5e0ce95c1959/7a043766-a0c2-4407-9464-91c0fba921a3"
-					(reference "R29")
+					(reference "R52")
 					(unit 1)
 				)
@@
 		(in_pos_files yes)
 		(dnp no)
-		(property "Reference" "R30"
+		(property "Reference" "R53"
 			(at 182.88 80.01 90)
 			(show_name no)
@@
 			(project "MIKA"
 				(path "/66ea9e27-3ca5-4edd-a0db-1f3995e73e78/c2d6fcaf-19aa-4c33-838f-5e0ce95c1959/7a043766-a0c2-4407-9464-91c0fba921a3"
-					(reference "R30")
+					(reference "R53")
 					(unit 1)
 				)
